File: Electronics/Full Adder/Design/Design.kicad_sch (KiCad schematic)
At the start: 0 parts

Commit message: completed the schematics of the full adder.
Parts:
- added U1: 74AUC2G86, symbol 74xGxx:74AUC2G86
- added U2: 74AUC2G08, symbol 74xGxx:74AUC2G08
- added U3: 74AUC2G32, symbol 74xGxx:74AUC2G32
Connections:
- new net: U1.5, U1.7, U2.6
- new net: U2.7, U3.2
- new net: U2.3, U3.1
- new net A: U1.1, U2.2
- new net B: U1.2, U2.1
- new net C: U1.6, U2.5
- new net Carry: U3.7
- new net Sum: U1.3

Commit message: finalized the footprints, to begin pcb design.
Parts:
- U1, U2, U3: footprint (none) -> Package_SO:SSOP-8_3.95x5.21x3.27mm_P1.27mm
Changed lines of the file:
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@@
 			)
 		)
-		(property "Footprint" ""
+		(property "Footprint" "Package_SO:SSOP-8_3.95x5.21x3.27mm_P1.27mm"
 			(at 201.93 73.66 0)
 			(hide yes)
@@
 			)
 		)
-		(property "Footprint" ""
+		(property "Footprint" "Package_SO:SSOP-8_3.95x5.21x3.27mm_P1.27mm"
 			(at 120.65 100.33 0)
 			(hide yes)
@@
 			)
 		)
-		(property "Footprint" ""
+		(property "Footprint" "Package_SO:SSOP-8_3.95x5.21x3.27mm_P1.27mm"
 			(at 200.66 93.98 0)
 			(hide yes)
@@
 			)
 		)
-		(property "Footprint" ""
+		(property "Footprint" "Package_SO:SSOP-8_3.95x5.21x3.27mm_P1.27mm"
 			(at 148.59 139.7 0)
 			(hide yes)
@@
 			)
 		)
-		(property "Footprint" ""
+		(property "Footprint" "Package_SO:SSOP-8_3.95x5.21x3.27mm_P1.27mm"
 			(at 179.07 139.7 0)
 			(hide yes)
@@
 			)
 		)
-		(property "Footprint" ""
+		(property "Footprint" "Package_SO:SSOP-8_3.95x5.21x3.27mm_P1.27mm"
 			(at 123.19 71.12 0)
 			(hide yes)
@@
 			)
 		)
-		(property "Footprint" ""
+		(property "Footprint" "Package_SO:SSOP-8_3.95x5.21x3.27mm_P1.27mm"
 			(at 173.99 91.44 0)
 			(hide yes)
@@
 			)
 		)
-		(property "Footprint" ""
+		(property "Footprint" "Package_SO:SSOP-8_3.95x5.21x3.27mm_P1.27mm"
 			(at 118.11 139.7 0)
 			(hide yes)
